Commit message: Almost has unique naming in xacro. Just battling the hector_quadrotor tags

File: cvg_sim_gazebo/urdf/quadrotor.urdf.xacro (robot description, xacro)
@@ -3,9 +3,10 @@
     xmlns:sensor="http://playerstage.sourceforge.net/gazebo/xmlschema/#sensor"
     xmlns:controller="http://playerstage.sourceforge.net/gazebo/xmlschema/#controller"
-    xmlns:interface="http://playerstage.sourceforge.net/gazebo/xmlschema/#interface"
-    xmlns:xacro="http://playerstage.sourceforge.net/gazebo/xmlschema/#interface">
+    xmlns:interface="http://ros.org/wiki/xacro"
+    xmlns:xacro="http://ros.org/wiki/xacro">
+    <xacro:arg name="prefix" default="quadrotor"/>
     <!-- Included URDF Files -->
     <xacro:include filename="$(find cvg_sim_gazebo)/urdf/quadrotor_base.urdf.xacro" />
-    <!-- Instantiate quadrotor_base_macro once (has no parameters atm) -->
-    <quadrotor_base_macro />
+    <!-- Instantiate quadrotor_base_macro with the required parameters -->
+    <quadrotor_base_macro prefix="$(arg prefix)"/>
 </robot>

File: cvg_sim_gazebo/urdf/quadrotor_base.urdf.xacro (robot description, xacro)
@@ -2,12 +2,13 @@
 <robot xmlns:sensor="http://playerstage.sourceforge.net/gazebo/xmlschema/#sensor"
 xmlns:controller="http://playerstage.sourceforge.net/gazebo/xmlschema/#controller"
-xmlns:interface="http://playerstage.sourceforge.net/gazebo/xmlschema/#interface"
+xmlns:interface="http://ros.org/wiki/xacro"
 xmlns:xacro="http://ros.org/wiki/xacro"
 >
+  <xacro:arg name="prefix" default="quadrotor"/>
   <xacro:include filename="$(find cvg_sim_gazebo_plugins)/urdf/quadrotor_plugins.urdf.xacro" />
-  <property name="pi" value="3.1415926535897931" />
+  <!--<xacro:property name="pi" value="3.1415926535897931" />-->
   <!-- Main quadrotor link -->
-  <xacro:macro name="quadrotor_base_macro">
-    <link name="base_link">
+  <xacro:macro name="quadrotor_base_macro" params="prefix">
+    <link name="${prefix}_base_link">
       <visual>
         <origin xyz="0 0 0" rpy="0 0 0" />
@@ -23,5 +24,5 @@
       </collision>
     </link>
-    <link name="dummy_link">
+    <link name="${prefix}_dummy_link">
 	      <inertial>
         	<mass value="0.436" /> <!--value="1.477" />-->
@@ -32,13 +33,13 @@
       	      </inertial>
     </link>
-    <joint name="dummy_joint" type="fixed">
- 	 <parent link="base_link"/>
-         <child link="dummy_link"/>
+    <joint name="${prefix}_dummy_joint" type="fixed">
+ 	        <parent link="${prefix}_base_link"/>
+          <child link="${prefix}_dummy_link"/>
     </joint>
-    <gazebo reference="base_link">
+    <gazebo reference="${prefix}_base_link">
       <turnGravityOff>false</turnGravityOff>
     </gazebo>
     <!-- Gazebo Plugins -->
-    <quadrotor_plugins/>
+    <quadrotor_plugins prefix="${prefix}"/>
   </xacro:macro>
 </robot>

File: cvg_sim_gazebo/urdf/quadrotor_sensors.urdf.xacro (robot description, xacro)
@@ -3,7 +3,7 @@
 xmlns:sensor="http://playerstage.sourceforge.net/gazebo/xmlschema/#sensor"
 xmlns:controller="http://playerstage.sourceforge.net/gazebo/xmlschema/#controller"
-xmlns:interface="http://playerstage.sourceforge.net/gazebo/xmlschema/#interface"
-xmlns:xacro="http://playerstage.sourceforge.net/gazebo/xmlschema/#interface">
-    <property name="M_PI" value="3.1415926535897931" />
+xmlns:interface="http://ros.org/wiki/xacro"
+xmlns:xacro="http://ros.org/wiki/xacro">
+    <xacro:property name="M_PI" value="3.1415926535897931" />
     <!-- Included URDF Files -->
     <xacro:include filename="$(find cvg_sim_gazebo)/urdf/quadrotor_base.urdf.xacro" />

File: cvg_sim_gazebo/urdf/sensors/generic_camera.urdf.xacro (robot description, xacro)
@@ -2,11 +2,11 @@
 <robot xmlns:sensor="http://playerstage.sourceforge.net/gazebo/xmlschema/#sensor"
 xmlns:controller="http://playerstage.sourceforge.net/gazebo/xmlschema/#controller"
-xmlns:interface="http://playerstage.sourceforge.net/gazebo/xmlschema/#interface"
+xmlns:interface="http://ros.org/wiki/xacro"
   xmlns:xacro="http://ros.org/wiki/xacro"
   >
-    <property name="M_PI" value="3.1415926535897931" />
+    <xacro:property name="M_PI" value="3.1415926535897931" />
     <xacro:macro name="generic_camera" params="name sim_name parent *origin update_rate res_x res_y image_format hfov">
       <joint name="${name}_joint" type="fixed">
-        <insert_block name="origin" />
+        <xacro:insert_block name="origin" />
         <parent link="${parent}"/>
         <child link="${name}_link"/>

File: cvg_sim_gazebo/urdf/sensors/hokuyo_utm30lx.urdf.xacro (robot description, xacro)
@@ -2,10 +2,10 @@
 <robot xmlns:sensor="http://playerstage.sourceforge.net/gazebo/xmlschema/#sensor"
 xmlns:controller="http://playerstage.sourceforge.net/gazebo/xmlschema/#controller"
-xmlns:interface="http://playerstage.sourceforge.net/gazebo/xmlschema/#interface"
+xmlns:interface="http://ros.org/wiki/xacro"
   xmlns:xacro="http://ros.org/wiki/xacro"
   >
     <xacro:macro name="hokuyo_utm30lx" params="name parent *origin ros_topic update_rate ray_count min_angle max_angle">
       <joint name="${name}_joint" type="fixed">
-	<insert_block name="origin" />
+	<xacro:insert_block name="origin" />
 	<parent link="${parent}"/>
 	<child link="${name}_frame"/>

File: cvg_sim_gazebo/urdf/sensors/sonar_sensor.urdf.xacro (robot description, xacro)
@@ -2,5 +2,5 @@
 <robot xmlns:sensor="http://playerstage.sourceforge.net/gazebo/xmlschema/#sensor"
 xmlns:controller="http://playerstage.sourceforge.net/gazebo/xmlschema/#controller"
-xmlns:interface="http://playerstage.sourceforge.net/gazebo/xmlschema/#interface"
+xmlns:interface="http://ros.org/wiki/xacro"
 xmlns:xacro="http://ros.org/wiki/xacro"
 >

File: cvg_sim_gazebo_plugins/urdf/quadrotor_plugins.urdf.xacro (robot description, xacro)
@@ -1,11 +1,12 @@
 <?xml version="1.0"?>
 <robot xmlns:xacro="http://ros.org/wiki/xacro">
+  <xacro:arg name="prefix" default="quadrotor"/>
   <xacro:include filename="$(find cvg_sim_gazebo_plugins)/urdf/quadrotor_sensors.urdf.xacro" />
   <xacro:include filename="$(find cvg_sim_gazebo_plugins)/urdf/quadrotor_simple_controller.urdf.xacro" />
   <!-- Quadrotor Gazebo Plugins -->
-  <xacro:macro name="quadrotor_plugins">
-    <canonicalBody>base_link</canonicalBody>
-    <quadrotor_sensors/>
-    <quadrotor_controller/>
+  <xacro:macro name="quadrotor_plugins" params="prefix">
+    <canonicalBody value="${prefix}_base_link"></canonicalBody>
+    <quadrotor_sensors prefix="${prefix}"/>
+    <quadrotor_controller prefix="${prefix}"/>
   </xacro:macro>
 </robot>

File: cvg_sim_gazebo_plugins/urdf/quadrotor_sensors.urdf.xacro (robot description, xacro)
@@ -2,17 +2,18 @@
 <robot xmlns:sensor="http://playerstage.sourceforge.net/gazebo/xmlschema/#sensor"
 xmlns:controller="http://playerstage.sourceforge.net/gazebo/xmlschema/#controller"
-xmlns:interface="http://playerstage.sourceforge.net/gazebo/xmlschema/#interface"
+xmlns:interface="http://ros.org/wiki/xacro"
 xmlns:xacro="http://ros.org/wiki/xacro"
 >
+<xacro:arg name="prefix" default="quadrotor"/>
   <!-- Quadrotor Sensor Plugins
         <frameId>ardrone_base_link</frameId>
 -->
-  <xacro:macro name="quadrotor_sensors">
+  <xacro:macro name="quadrotor_sensors" params="prefix">
     <gazebo>
       <plugin name="quadrotor_imu_sim" filename="libhector_gazebo_ros_imu.so">
         <alwaysOn>true</alwaysOn>
         <updateRate>100.0</updateRate>
-        <bodyName>base_link</bodyName>
-        <frameId>ardrone_base_link</frameId>
+        <bodyName value="${prefix}_base_link"></bodyName>
+        <frameId value="${prefix}_ardrone_base_link"></frameId>
         <topicName>ardrone/imu</topicName>
         <rpyOffsets>0 0 0</rpyOffsets> <!-- deprecated -->
@@ -34,5 +35,5 @@
         <alwaysOn>true</alwaysOn>
         <updateRate>10.0</updateRate>
-        <bodyName>base_link</bodyName>
+        <bodyName value="${prefix}_base_link"></bodyName>
         <topicName>pressure_height</topicName>
         <altimeterTopicName>altimeter</altimeterTopicName>
@@ -45,5 +46,5 @@
         <alwaysOn>true</alwaysOn>
         <updateRate>10.0</updateRate>
-        <bodyName>base_link</bodyName>
+        <bodyName value="${prefix}_base_link"></bodyName>
         <topicName>magnetic</topicName>
         <offset>0 0 0</offset>
@@ -55,5 +56,5 @@
         <alwaysOn>true</alwaysOn>
         <updateRate>4.0</updateRate>
-        <bodyName>base_link</bodyName>
+        <bodyName value="${prefix}_base_link"></bodyName>
         <topicName>fix</topicName>
         <velocityTopicName>fix_velocity</velocityTopicName>
@@ -70,5 +71,5 @@
         <alwaysOn>true</alwaysOn>
         <updateRate>100.0</updateRate>
-        <bodyName>base_link</bodyName>
+        <bodyName value="${prefix}_base_link"></bodyName>
         <topicName>ground_truth/state</topicName>
         <gaussianNoise>0.0</gaussianNoise>

File: cvg_sim_gazebo_plugins/urdf/quadrotor_simple_controller.urdf.xacro (robot description, xacro)
@@ -4,17 +4,16 @@
 xmlns:xacro="http://ros.org/wiki/xacro"
 >
+<xacro:arg name="prefix" default="quadrotor"/>
   <!-- Quadrotor Simple Controller Plugin -->
-  <xacro:macro name="quadrotor_controller">
+  <xacro:macro name="quadrotor_controller" params="prefix">
     <gazebo>
       <plugin name="quadrotor_simple_controller" filename="libhector_gazebo_quadrotor_simple_controller.so">
         <alwaysOn>true</alwaysOn>
         <updateRate>0.0</updateRate>
-        <bodyName>base_link</bodyName>
+        <bodyName value="${prefix}_base_link"></bodyName>
         <stateTopic>ground_truth/state</stateTopic>
         <imuTopic>ardrone/imu</imuTopic>
         <navdataTopic>ardrone/navdata</navdataTopic>
         <resetTopic>ardrone/reset</resetTopic>
-        <!--<takeoffTopic>ardrone/takeoff</takeoffTopic>
-        <landTopic>ardrone/land</landTopic>-->
         <topicName>cmd_vel</topicName>
         <rollpitchProportionalGain>10.0</rollpitchProportionalGain>
@@ -38,5 +37,5 @@
         <alwaysOn>true</alwaysOn>
         <updateRate>0.0</updateRate>
-        <bodyName>base_link</bodyName>
+        <bodyName value="${prefix}_base_link"></bodyName>
         <stateTopic>ground_truth/state</stateTopic>
         <imuTopic>ardrone/imu</imuTopic>
