Commit message: Aligns drone weight and inertia with real values

File: cvg_sim_gazebo/urdf/quadrotor_base.urdf.xacro (robot description, xacro)
@@ -25,7 +25,9 @@
     <link name="dummy_link">
 	      <inertial>
-        	<mass value="1.477" />
+        	<mass value="0.436" /> <!--value="1.477" />-->
         	<origin xyz="0 0 0" />
-        	<inertia ixx="0.01152" ixy="0.0" ixz="0.0" iyy="0.01152" iyz="0.0" izz="0.0218" />
+        	<!--<inertia ixx="0.01152" ixy="0.0" ixz="0.0" iyy="0.01152" iyz="0.0" izz="0.0218" />-->
+          <!-- <inertia ixx="0.0347563" ixy="0.0" ixz="0.0" iyy="0.0458929" iyz="0.0" izz="0.0977" /> -->
+          <inertia ixx="0.045" ixy="0.0" ixz="0.0" iyy="0.051" iyz="0.0" izz="0.095" />
       	      </inertial>
     </link>

Commit message: Makes inertia values of drone correct

File: cvg_sim_gazebo/urdf/quadrotor_base.urdf.xacro (robot description, xacro)
@@ -29,5 +29,5 @@
         	<!--<inertia ixx="0.01152" ixy="0.0" ixz="0.0" iyy="0.01152" iyz="0.0" izz="0.0218" />-->
           <!-- <inertia ixx="0.0347563" ixy="0.0" ixz="0.0" iyy="0.0458929" iyz="0.0" izz="0.0977" /> -->
-          <inertia ixx="0.045" ixy="0.0" ixz="0.0" iyy="0.051" iyz="0.0" izz="0.095" />
+          <inertia ixx="0.0045" ixy="0.0" ixz="0.0" iyy="0.0051" iyz="0.0" izz="0.0095" />
       	      </inertial>
     </link>

Commit message: Fixes infinite hover by not paying attention to the sonar

File: cvg_sim_gazebo/urdf/quadrotor_base.urdf.xacro (robot description, xacro)
@@ -31,5 +31,5 @@
           <!-- <inertia ixx="0.0347563" ixy="0.0" ixz="0.0" iyy="0.0458929" iyz="0.0" izz="0.0977" /> -->
           <inertia ixx="0.0045" ixy="0.0" ixz="0.0" iyy="0.0051" iyz="0.0" izz="0.0095" />
-      	      </inertial>
+      	</inertial>
     </link>
     <joint name="${prefix}_dummy_joint" type="fixed">

File: cvg_sim_gazebo_plugins/urdf/quadrotor_sensors.urdf.xacro (robot description, xacro)
@@ -76,4 +76,9 @@
         <frameName>map</frameName>
       </plugin>
+      <!-- Sonar height sensor
+      <plugin name="quadrotor_sonar_sim" filename="libhector_gazebo_ros_sonar.so">
+        <bodyName>${prefix}_base_link</bodyName>
+        <topicName>sonar_height</topicName>
+      </plugin>-->
     </gazebo>
   </xacro:macro>

File: cvg_sim_gazebo_plugins/urdf/quadrotor_simple_controller.urdf.xacro (robot description, xacro)
@@ -40,5 +40,5 @@
         <stateTopic>ground_truth/state</stateTopic>
         <imuTopic>ardrone/imu</imuTopic>
-        <sonarTopic>sonar_height</sonarTopic>
+        <!--<sonarTopic>sonar_height</sonarTopic>-->
         <topicName>cmd_vel</topicName>
         <navdataTopic>ardrone/navdata</navdataTopic>
